File: FeroFly.kicad_sch (KiCad schematic)
At the start: 0 parts

Commit message: feat: add mounting holes
Parts:
- added H101, H102, H103, H104: MountingHole, MountingHole:MountingHole_3.2mm_M3, symbol Mechanical:MountingHole
Other:
- note added: "M3 Mounting Holes"
