File: FeroFly.kicad_pcb (KiCad board)
At the start: 2 copper layers, 149 parts, among them J301 Conn_01x04_Pin, J601 SM04B-GHS-TB(LF)(SN), J801 SM04B-GHS-TB(LF)(SN), J802 SM06B-GHS-TB(LF)(SN), J803 SM04B-GHS-TB(LF)(SN), J804 SM04B-GHS-TB(LF)(SN), J805 SM06B-GHS-TB(LF)(SN), J901 Conn_01x03_Pin, J902 Conn_01x03_Pin, J903 Conn_01x03_Pin, J904 Conn_01x03_Pin, J905 Conn_01x03_Pin, J906 Conn_01x03_Pin, J907 Conn_01x03_Pin, J908 Conn_01x03_Pin, J909 Conn_01x03_Pin, J910 Conn_01x03_Pin, J911 Conn_01x03_Pin, J912 Conn_01x03_Pin, J913 12402012E212A, J914 SM04B-GHS-TB(LF)(SN), SW301 SW_Push, SW302 SW_Push, U201 AP62200WU-7, U202 TLV75733PDRV, U301 STM32F405RGTx, U501 LSM6DSL, U502 BMP390, U601 SN65HVD230DR, U901 USBLC6-2P6, Y301 24MHz

Commit message: feat: add mounting holes
Parts:
- added H101: MountingHole, MountingHole:MountingHole_3.2mm_M3, F.Cu at (187.7, 78.2)
- added H102: MountingHole, MountingHole:MountingHole_3.2mm_M3, F.Cu at (187.7, 86.1)
- added H103: MountingHole, MountingHole:MountingHole_3.2mm_M3, F.Cu at (187.7, 94.1)
- added H104: MountingHole, MountingHole:MountingHole_3.2mm_M3, F.Cu at (187.7, 102.0)

Commit message: feat: add layout notes and net labels
Parts:
- R605: footprint Resistor_SMD:R_0603_1608Metric_Pad0.98x0.95mm_HandSolder -> Resistor_SMD:R_1206_3216Metric_Pad1.30x1.75mm_HandSolder
Connections:
- net Net-(J601-Pin_2) renamed /Peripherals/CAN & LEDs/CAN+
- net Net-(J601-Pin_3) renamed /Peripherals/CAN & LEDs/CAN-
Changed lines of the file:
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@@
 			(layers "F.Cu" "F.Mask" "F.Paste")
 			(roundrect_rratio 0.25)
-			(net "Net-(J601-Pin_3)")
+			(net "/Peripherals/CAN & LEDs/CAN-")
 			(pinfunction "K_1")
 			(pintype "passive")
@@
 			(layers "F.Cu" "F.Mask" "F.Paste")
 			(roundrect_rratio 0.25)
-			(net "Net-(J601-Pin_2)")
+			(net "/Peripherals/CAN & LEDs/CAN+")
 			(pinfunction "K_2")
 			(pintype "passive")
@@
 			(layers "F.Cu" "F.Mask" "F.Paste")
 			(roundrect_rratio 0.25)
-			(net "Net-(J601-Pin_3)")
+			(net "/Peripherals/CAN & LEDs/CAN-")
 			(pinfunction "CANL_6")
 			(pintype "bidirectional")
@@
 			(layers "F.Cu" "F.Mask" "F.Paste")
 			(roundrect_rratio 0.25)
-			(net "Net-(J601-Pin_2)")
+			(net "/Peripherals/CAN & LEDs/CAN+")
 			(pinfunction "CANH_7")
 			(pintype "bidirectional")
@@
 			(layers "F.Cu" "F.Mask" "F.Paste")
 			(roundrect_rratio 0.25)
-			(net "Net-(J601-Pin_2)")
+			(net "/Peripherals/CAN & LEDs/CAN+")
 			(pinfunction "Pin_2_2")
 			(pintype "passive")
@@
 			(layers "F.Cu" "F.Mask" "F.Paste")
 			(roundrect_rratio 0.25)
-			(net "Net-(J601-Pin_3)")
+			(net "/Peripherals/CAN & LEDs/CAN-")
 			(pinfunction "Pin_3_3")
 			(pintype "passive")
@@
 			(size 0.3 0.3)
 			(layers "F.Cu" "F.Mask")
-			(net "Net-(J601-Pin_2)")
+			(net "/Peripherals/CAN & LEDs/CAN+")
 			(pinfunction "A_1")
 			(pintype "passive")
@@
 		)
 	)
-	(footprint "Resistor_SMD:R_0603_1608Metric_Pad0.98x0.95mm_HandSolder"
+	(footprint "Resistor_SMD:R_1206_3216Metric_Pad1.30x1.75mm_HandSolder"
 		(layer "F.Cu")
 		(at 118.275 134.115)
-		(descr "Resistor SMD 0603 (1608 Metric), square (rectangular) end terminal, IPC-7351 nominal with elongated pad for handsoldering. (Body size source: IPC-SM-782 page 72, https://www.pcb-3d.com/wordpress/wp-content/uploads/ipc-sm-782a_amendment_1_and_2.pdf)")
+		(descr "Resistor SMD 1206 (3216 Metric), square (rectangular) end terminal, IPC-7351 nominal with elongated pad for handsoldering. (Body size source: IPC-SM-782 page 72, https://www.pcb-3d.com/wordpress/wp-content/uploads/ipc-sm-782a_amendment_1_and_2.pdf)")
 		(tags "resistor handsolder")
 		(property "Reference" "R605"
-			(at 0 -1.43 0)
+			(at 0 -1.83 0)
 			(layer "F.SilkS")
 			(effects
@@
 		)
 		(property "Value" "120"
-			(at 0 1.43 0)
+			(at 0 1.83 0)
 			(layer "F.Fab")
 			(effects
@@
 			)
 		)
-		(property "MPN" "CR0603-FX-1200ELF"
+		(property "MPN" "CR1206-FX-1200ELF"
 			(at 0 0 0)
 			(unlocked yes)
@@
 			)
 		)
-		(property "MANUFACTURER" ""
-			(at 0 0 0)
-			(unlocked yes)
-			(layer "F.Fab")
-			(hide yes)
-			(effects
-				(font
-					(size 1 1)
-					(thickness 0.15)
-				)
-			)
-		)
-		(property "KLC_S3.3" ""
-			(at 0 0 0)
-			(unlocked yes)
-			(layer "F.Fab")
-			(hide yes)
-			(effects
-				(font
-					(size 1 1)
-					(thickness 0.15)
-				)
-			)
-		)
-		(property "KLC_S4.1" ""
-			(at 0 0 0)
-			(unlocked yes)
-			(layer "F.Fab")
-			(hide yes)
-			(effects
-				(font
-					(size 1 1)
-					(thickness 0.15)
-				)
-			)
-		)
 		(property ki_fp_filters "R_*")
 		(sheetname "/Peripherals/CAN & LEDs/")
@@
 		(duplicate_pad_numbers_are_jumpers no)
 		(fp_line
-			(start -0.254724 -0.5225)
-			(end 0.254724 -0.5225)
+			(start -0.727064 -0.91)
+			(end 0.727064 -0.91)
 			(stroke
 				(width 0.12)
@@
 		)
 		(fp_line
-			(start -0.254724 0.5225)
-			(end 0.254724 0.5225)
+			(start -0.727064 0.91)
+			(end 0.727064 0.91)
 			(stroke
 				(width 0.12)
@@
 		)
 		(fp_rect
-			(start -1.65 -0.73)
-			(end 1.65 0.73)
+			(start -2.45 -1.13)
+			(end 2.45 1.13)
 			(stroke
 				(width 0.05)
@@
 		)
 		(fp_rect
-			(start -0.8 -0.4125)
-			(end 0.8 0.4125)
+			(start -1.6 -0.8)
+			(end 1.6 0.8)
 			(stroke
 				(width 0.1)
@@
 			(effects
 				(font
-					(size 0.4 0.4)
-					(thickness 0.06)
+					(size 0.8 0.8)
+					(thickness 0.12)
 				)
 			)
 		)
 		(pad "1" smd roundrect
-			(at -0.9125 0)
-			(size 0.975 0.95)
+			(at -1.55 0)
+			(size 1.3 1.75)
 			(layers "F.Cu" "F.Mask" "F.Paste")
-			(roundrect_rratio 0.25)
+			(roundrect_rratio 0.192308)
 			(net "Net-(JP601-B)")
 			(pintype "passive")
 		)
 		(pad "2" smd roundrect
-			(at 0.9125 0)
-			(size 0.975 0.95)
+			(at 1.55 0)
+			(size 1.3 1.75)
 			(layers "F.Cu" "F.Mask" "F.Paste")
-			(roundrect_rratio 0.25)
-			(net "Net-(J601-Pin_3)")
+			(roundrect_rratio 0.192308)
+			(net "/Peripherals/CAN & LEDs/CAN-")
 			(pintype "passive")
 		)
 		(embedded_fonts no)
-		(model "${KICAD10_3DMODEL_DIR}/Resistor_SMD.3dshapes/R_0603_1608Metric.step"
+		(model "${KICAD10_3DMODEL_DIR}/Resistor_SMD.3dshapes/R_1206_3216Metric.step"
 			(offset
 				(xyz 0 0 0)
