File: Peripherals.kicad_sch (KiCad schematic)
At the start: 0 parts

Commit message: refactor: change name from FeroFly405 to FeroFlyF405
Other:
- title: FeroFly405 -> FeroFlyF405
Changed lines of the file:
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@@
 	(paper "A4")
 	(title_block
-		(title "FeroFly405")
+		(title "FeroFlyF405")
 		(date "2026-07-22")
 		(rev "1")
-		(comment 3 "GitHub: https://github.com/Ozonised/FeroFly405")
+		(comment 3 "GitHub: https://github.com/Ozonised/FeroFlyF405")
 		(comment 4 "Designed by: Farhan Khan")
 	)
@@
 		)
 		(instances
-			(project "FeroFly"
+			(project "FeroFlyF405"
 				(path "/8fea5468-8d8d-4bdb-afc0-e65b62c92669/2db1372a-2ed6-420c-af8b-d4f9c1346569"
 					(page "6")
@@
 		)
 		(instances
-			(project "FeroFly"
+			(project "FeroFlyF405"
 				(path "/8fea5468-8d8d-4bdb-afc0-e65b62c92669/2db1372a-2ed6-420c-af8b-d4f9c1346569"
 					(page "5")

Commit message: refactor(schematic): assign net classes and fix USB net label assingment
Other:
- sheet IMUs ports: added SPI1_CS, SPI1_MISO, SPI1_MOSI, SPI1_SCK; removed D_SPI1_CS, D_SPI1_MISO, D_SPI1_MOSI, D_SPI1_SCK
Changed lines of the file:
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@@
 		)
 	)
-	(hierarchical_label "D_SPI1_SCK"
+	(hierarchical_label "SPI1_SCK"
 		(shape output)
 		(at 53.34 97.79 180)
@@
 		)
 	)
-	(hierarchical_label "D_SPI1_CS"
+	(hierarchical_label "SPI1_CS"
 		(shape output)
 		(at 53.34 90.17 180)
@@
 		)
 	)
-	(hierarchical_label "D_SPI1_MOSI"
+	(hierarchical_label "SPI1_MOSI"
 		(shape output)
 		(at 53.34 95.25 180)
@@
 		)
 	)
-	(hierarchical_label "D_SPI1_MISO"
+	(hierarchical_label "SPI1_MISO"
 		(shape input)
 		(at 53.34 92.71 180)
@@
 			)
 		)
-		(pin "D_SPI1_CS" output
+		(pin "SPI1_CS" output
 			(at 67.31 90.17 180)
 			(effects
@@
 			)
 		)
-		(pin "D_SPI1_MISO" input
+		(pin "SPI1_MISO" input
 			(at 67.31 92.71 180)
 			(effects
@@
 			)
 		)
-		(pin "D_SPI1_MOSI" input
+		(pin "SPI1_MOSI" input
 			(at 67.31 95.25 180)
 			(effects
@@
 			)
 		)
-		(pin "D_SPI1_SCK" output
+		(pin "SPI1_SCK" output
 			(at 67.31 97.79 180)
 			(effects
