File: IO.kicad_sch (KiCad schematic)
At the start: 0 parts

Commit message: refactor: change name from FeroFly405 to FeroFlyF405
Other:
- title: FeroFly405 -> FeroFlyF405
Changed lines of the file:
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@@
 	(paper "A4")
 	(title_block
-		(title "FeroFly405")
+		(title "FeroFlyF405")
 		(date "2026-07-22")
 		(rev "1")
-		(comment 3 "GitHub: https://github.com/Ozonised/FeroFly405")
+		(comment 3 "GitHub: https://github.com/Ozonised/FeroFlyF405")
 		(comment 4 "Designed by: Farhan Khan")
 	)
@@
 		)
 		(instances
-			(project "FeroFly"
+			(project "FeroFlyF405"
 				(path "/8fea5468-8d8d-4bdb-afc0-e65b62c92669/eeef3184-c704-411c-8c4e-6f902313c1c6"
 					(page "9")
@@
 		)
 		(instances
-			(project "FeroFly"
+			(project "FeroFlyF405"
 				(path "/8fea5468-8d8d-4bdb-afc0-e65b62c92669/eeef3184-c704-411c-8c4e-6f902313c1c6"
 					(page "8")

Commit message: refactor: change motor output, renamed power nets
Other:
- sheet IO2 ports: added D_ADC1_CH10; removed D_ADC2_CH12
Changed lines of the file:
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@@
 		)
 	)
-	(hierarchical_label "D_ADC2_CH12"
+	(hierarchical_label "D_ADC1_CH10"
 		(shape input)
 		(at 195.58 132.08 180)
@@
 			)
 		)
-		(pin "D_ADC2_CH12" input
+		(pin "D_ADC1_CH10" input
 			(at 201.93 124.46 270)
 			(effects
