File: IO.kicad_sch (KiCad schematic)
At the start: 0 parts

Commit message: refactor: change tim5 ch 1 label to ch 2
Changed lines of the file:
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@@
 		)
 	)
-	(hierarchical_label "D_TIM5_CH1"
+	(hierarchical_label "D_TIM5_CH2"
 		(shape bidirectional)
 		(at 171.45 110.49 180)

Commit message: fix!: change ouput 3 timer from tim4 ch4 to tim1 ch3
tim4 ch4 does not have dma. Therefore replaced it with tim1 ch3.
Other:
- sheet IO2 ports: added D_TIM1_CH3; removed D_TIM4_CH4
Changed lines of the file:
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@@
 		(title "FeroFlyF405")
 		(date "2026-07-22")
-		(rev "1")
+		(rev "1.1")
 		(comment 2 "LICENSE: CERN-OHL-S-2.0 ")
 		(comment 3 "GitHub: https://github.com/Ozonised/FeroFlyF405")
@@
 		)
 	)
-	(hierarchical_label "D_TIM4_CH4"
+	(hierarchical_label "D_TIM1_CH3"
 		(shape bidirectional)
 		(at 171.45 107.95 180)
@@
 			)
 		)
-		(pin "D_TIM4_CH4" bidirectional
+		(pin "D_TIM1_CH3" bidirectional
 			(at 179.07 107.95 180)
 			(effects
