File: IO1.kicad_sch (KiCad schematic)
At the start: 25 parts, among them J801 SM04B-GHS-TB(LF)(SN), J802 SM06B-GHS-TB(LF)(SN), J803 SM04B-GHS-TB(LF)(SN), J804 SM04B-GHS-TB(LF)(SN), J805 SM06B-GHS-TB(LF)(SN)

Commit message: refactor: change name from FeroFly405 to FeroFlyF405
Other:
- title: FeroFly405 -> FeroFlyF405
Changed lines of the file:
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@@
 	(paper "A4")
 	(title_block
-		(title "FeroFly405")
+		(title "FeroFlyF405")
 		(date "2026-07-22")
 		(rev "1")
-		(comment 3 "GitHub: https://github.com/Ozonised/FeroFly405")
+		(comment 3 "GitHub: https://github.com/Ozonised/FeroFlyF405")
 		(comment 4 "Designed by: Farhan Khan")
 	)
@@
 		)
 		(instances
-			(project "FeroFly"
+			(project "FeroFlyF405"
 				(path "/8fea5468-8d8d-4bdb-afc0-e65b62c92669/eeef3184-c704-411c-8c4e-6f902313c1c6/999244e6-4bab-413b-b198-56b8312054d8"
 					(reference "TP802")
@@
 		)
 		(instances
-			(project "FeroFly"
+			(project "FeroFlyF405"
 				(path "/8fea5468-8d8d-4bdb-afc0-e65b62c92669/eeef3184-c704-411c-8c4e-6f902313c1c6/999244e6-4bab-413b-b198-56b8312054d8"
 					(reference "TP809")
@@
 		)
 		(instances
-			(project "FeroFly"
+			(project "FeroFlyF405"
 				(path "/8fea5468-8d8d-4bdb-afc0-e65b62c92669/eeef3184-c704-411c-8c4e-6f902313c1c6/999244e6-4bab-413b-b198-56b8312054d8"
 					(reference "J804")
@@
 		)
 		(instances
-			(project "FeroFly"
+			(project "FeroFlyF405"
 				(path "/8fea5468-8d8d-4bdb-afc0-e65b62c92669/eeef3184-c704-411c-8c4e-6f902313c1c6/999244e6-4bab-413b-b198-56b8312054d8"
 					(reference "#PWR0806")
@@
 		)
 		(instances
-			(project "FeroFly"
+			(project "FeroFlyF405"
 				(path "/8fea5468-8d8d-4bdb-afc0-e65b62c92669/eeef3184-c704-411c-8c4e-6f902313c1c6/999244e6-4bab-413b-b198-56b8312054d8"
 					(reference "TP815")
@@
 		)
 		(instances
-			(project "FeroFly"
+			(project "FeroFlyF405"
 				(path "/8fea5468-8d8d-4bdb-afc0-e65b62c92669/eeef3184-c704-411c-8c4e-6f902313c1c6/999244e6-4bab-413b-b198-56b8312054d8"
 					(reference "TP807")
@@
 		)
 		(instances
-			(project "FeroFly"
+			(project "FeroFlyF405"
 				(path "/8fea5468-8d8d-4bdb-afc0-e65b62c92669/eeef3184-c704-411c-8c4e-6f902313c1c6/999244e6-4bab-413b-b198-56b8312054d8"
 					(reference "#PWR0812")
@@
 		)
 		(instances
-			(project "FeroFly"
+			(project "FeroFlyF405"
 				(path "/8fea5468-8d8d-4bdb-afc0-e65b62c92669/eeef3184-c704-411c-8c4e-6f902313c1c6/999244e6-4bab-413b-b198-56b8312054d8"
 					(reference "#PWR0802")
@@
 		)
 		(instances
-			(project "FeroFly"
+			(project "FeroFlyF405"
 				(path "/8fea5468-8d8d-4bdb-afc0-e65b62c92669/eeef3184-c704-411c-8c4e-6f902313c1c6/999244e6-4bab-413b-b198-56b8312054d8"
 					(reference "TP801")
@@
 		)
 		(instances
-			(project "FeroFly"
+			(project "FeroFlyF405"
 				(path "/8fea5468-8d8d-4bdb-afc0-e65b62c92669/eeef3184-c704-411c-8c4e-6f902313c1c6/999244e6-4bab-413b-b198-56b8312054d8"
 					(reference "#PWR0814")
@@
 		)
 		(instances
-			(project "FeroFly"
+			(project "FeroFlyF405"
 				(path "/8fea5468-8d8d-4bdb-afc0-e65b62c92669/eeef3184-c704-411c-8c4e-6f902313c1c6/999244e6-4bab-413b-b198-56b8312054d8"
 					(reference "TP803")
@@
 		)
 		(instances
-			(project "FeroFly"
+			(project "FeroFlyF405"
 				(path "/8fea5468-8d8d-4bdb-afc0-e65b62c92669/eeef3184-c704-411c-8c4e-6f902313c1c6/999244e6-4bab-413b-b198-56b8312054d8"
 					(reference "J801")
@@
 		)
 		(instances
-			(project "FeroFly"
+			(project "FeroFlyF405"
 				(path "/8fea5468-8d8d-4bdb-afc0-e65b62c92669/eeef3184-c704-411c-8c4e-6f902313c1c6/999244e6-4bab-413b-b198-56b8312054d8"
 					(reference "#PWR0808")
@@
 		)
 		(instances
-			(project "FeroFly"
+			(project "FeroFlyF405"
 				(path "/8fea5468-8d8d-4bdb-afc0-e65b62c92669/eeef3184-c704-411c-8c4e-6f902313c1c6/999244e6-4bab-413b-b198-56b8312054d8"
 					(reference "TP812")
@@
 		)
 		(instances
-			(project "FeroFly"
+			(project "FeroFlyF405"
 				(path "/8fea5468-8d8d-4bdb-afc0-e65b62c92669/eeef3184-c704-411c-8c4e-6f902313c1c6/999244e6-4bab-413b-b198-56b8312054d8"
 					(reference "TP804")
@@
 		)
 		(instances
-			(project "FeroFly"
+			(project "FeroFlyF405"
 				(path "/8fea5468-8d8d-4bdb-afc0-e65b62c92669/eeef3184-c704-411c-8c4e-6f902313c1c6/999244e6-4bab-413b-b198-56b8312054d8"
 					(reference "#PWR0811")
@@
 		)
 		(instances
-			(project "FeroFly"
+			(project "FeroFlyF405"
 				(path "/8fea5468-8d8d-4bdb-afc0-e65b62c92669/eeef3184-c704-411c-8c4e-6f902313c1c6/999244e6-4bab-413b-b198-56b8312054d8"
 					(reference "J803")
@@
 		)
 		(instances
-			(project "FeroFly"
+			(project "FeroFlyF405"
 				(path "/8fea5468-8d8d-4bdb-afc0-e65b62c92669/eeef3184-c704-411c-8c4e-6f902313c1c6/999244e6-4bab-413b-b198-56b8312054d8"
 					(reference "C803")
@@
 		)
 		(instances
-			(project "FeroFly"
+			(project "FeroFlyF405"
 				(path "/8fea5468-8d8d-4bdb-afc0-e65b62c92669/eeef3184-c704-411c-8c4e-6f902313c1c6/999244e6-4bab-413b-b198-56b8312054d8"
 					(reference "#PWR0804")
@@
 		)
 		(instances
-			(project "FeroFly"
+			(project "FeroFlyF405"
 				(path "/8fea5468-8d8d-4bdb-afc0-e65b62c92669/eeef3184-c704-411c-8c4e-6f902313c1c6/999244e6-4bab-413b-b198-56b8312054d8"
 					(reference "#PWR0803")
@@
 		)
 		(instances
-			(project "FeroFly"
+			(project "FeroFlyF405"
 				(path "/8fea5468-8d8d-4bdb-afc0-e65b62c92669/eeef3184-c704-411c-8c4e-6f902313c1c6/999244e6-4bab-413b-b198-56b8312054d8"
 					(reference "#PWR0813")
@@
 		)
 		(instances
-			(project "FeroFly"
+			(project "FeroFlyF405"
 				(path "/8fea5468-8d8d-4bdb-afc0-e65b62c92669/eeef3184-c704-411c-8c4e-6f902313c1c6/999244e6-4bab-413b-b198-56b8312054d8"
 					(reference "C802")
@@
 		)
 		(instances
-			(project "FeroFly"
+			(project "FeroFlyF405"
 				(path "/8fea5468-8d8d-4bdb-afc0-e65b62c92669/eeef3184-c704-411c-8c4e-6f902313c1c6/999244e6-4bab-413b-b198-56b8312054d8"
 					(reference "#PWR0807")
@@
 		)
 		(instances
-			(project "FeroFly"
+			(project "FeroFlyF405"
 				(path "/8fea5468-8d8d-4bdb-afc0-e65b62c92669/eeef3184-c704-411c-8c4e-6f902313c1c6/999244e6-4bab-413b-b198-56b8312054d8"
 					(reference "#PWR0801")
@@
 		)
 		(instances
-			(project "FeroFly"
+			(project "FeroFlyF405"
 				(path "/8fea5468-8d8d-4bdb-afc0-e65b62c92669/eeef3184-c704-411c-8c4e-6f902313c1c6/999244e6-4bab-413b-b198-56b8312054d8"
 					(reference "#PWR0810")
@@
 		)
 		(instances
-			(project "FeroFly"
+			(project "FeroFlyF405"
 				(path "/8fea5468-8d8d-4bdb-afc0-e65b62c92669/eeef3184-c704-411c-8c4e-6f902313c1c6/999244e6-4bab-413b-b198-56b8312054d8"
 					(reference "C804")
@@
 		)
 		(instances
-			(project "FeroFly"
+			(project "FeroFlyF405"
 				(path "/8fea5468-8d8d-4bdb-afc0-e65b62c92669/eeef3184-c704-411c-8c4e-6f902313c1c6/999244e6-4bab-413b-b198-56b8312054d8"
 					(reference "TP808")
@@
 		)
 		(instances
-			(project "FeroFly"
+			(project "FeroFlyF405"
 				(path "/8fea5468-8d8d-4bdb-afc0-e65b62c92669/eeef3184-c704-411c-8c4e-6f902313c1c6/999244e6-4bab-413b-b198-56b8312054d8"
 					(reference "TP810")
@@
 		)
 		(instances
-			(project "FeroFly"
+			(project "FeroFlyF405"
 				(path "/8fea5468-8d8d-4bdb-afc0-e65b62c92669/eeef3184-c704-411c-8c4e-6f902313c1c6/999244e6-4bab-413b-b198-56b8312054d8"
 					(reference "J802")
@@
 		)
 		(instances
-			(project "FeroFly"
+			(project "FeroFlyF405"
 				(path "/8fea5468-8d8d-4bdb-afc0-e65b62c92669/eeef3184-c704-411c-8c4e-6f902313c1c6/999244e6-4bab-413b-b198-56b8312054d8"
 					(reference "#PWR0805")
@@
 		)
 		(instances
-			(project "FeroFly"
+			(project "FeroFlyF405"
 				(path "/8fea5468-8d8d-4bdb-afc0-e65b62c92669/eeef3184-c704-411c-8c4e-6f902313c1c6/999244e6-4bab-413b-b198-56b8312054d8"
 					(reference "TP806")
@@
 		)
 		(instances
-			(project "FeroFly"
+			(project "FeroFlyF405"
 				(path "/8fea5468-8d8d-4bdb-afc0-e65b62c92669/eeef3184-c704-411c-8c4e-6f902313c1c6/999244e6-4bab-413b-b198-56b8312054d8"
 					(reference "J805")
@@
 		)
 		(instances
-			(project "FeroFly"
+			(project "FeroFlyF405"
 				(path "/8fea5468-8d8d-4bdb-afc0-e65b62c92669/eeef3184-c704-411c-8c4e-6f902313c1c6/999244e6-4bab-413b-b198-56b8312054d8"
 					(reference "TP813")
@@
 		)
 		(instances
-			(project "FeroFly"
+			(project "FeroFlyF405"
 				(path "/8fea5468-8d8d-4bdb-afc0-e65b62c92669/eeef3184-c704-411c-8c4e-6f902313c1c6/999244e6-4bab-413b-b198-56b8312054d8"
 					(reference "C805")
@@
 		)
 		(instances
-			(project "FeroFly"
+			(project "FeroFlyF405"
 				(path "/8fea5468-8d8d-4bdb-afc0-e65b62c92669/eeef3184-c704-411c-8c4e-6f902313c1c6/999244e6-4bab-413b-b198-56b8312054d8"
 					(reference "TP805")
@@
 		)
 		(instances
-			(project "FeroFly"
+			(project "FeroFlyF405"
 				(path "/8fea5468-8d8d-4bdb-afc0-e65b62c92669/eeef3184-c704-411c-8c4e-6f902313c1c6/999244e6-4bab-413b-b198-56b8312054d8"
 					(reference "#PWR0815")
@@
 		)
 		(instances
-			(project "FeroFly"
+			(project "FeroFlyF405"
 				(path "/8fea5468-8d8d-4bdb-afc0-e65b62c92669/eeef3184-c704-411c-8c4e-6f902313c1c6/999244e6-4bab-413b-b198-56b8312054d8"
 					(reference "TP814")
@@
 		)
 		(instances
-			(project "FeroFly"
+			(project "FeroFlyF405"
 				(path "/8fea5468-8d8d-4bdb-afc0-e65b62c92669/eeef3184-c704-411c-8c4e-6f902313c1c6/999244e6-4bab-413b-b198-56b8312054d8"
 					(reference "TP811")
@@
 		)
 		(instances
-			(project "FeroFly"
+			(project "FeroFlyF405"
 				(path "/8fea5468-8d8d-4bdb-afc0-e65b62c92669/eeef3184-c704-411c-8c4e-6f902313c1c6/999244e6-4bab-413b-b198-56b8312054d8"
 					(reference "C801")
@@
 		)
 		(instances
-			(project "FeroFly"
+			(project "FeroFlyF405"
 				(path "/8fea5468-8d8d-4bdb-afc0-e65b62c92669/eeef3184-c704-411c-8c4e-6f902313c1c6/999244e6-4bab-413b-b198-56b8312054d8"
 					(reference "#PWR0809")

Commit message: fix: silkcreen name guide and remove excess test points
Parts:
- removed TP801, TP803, TP807, TP808, TP810, TP811, TP813, TP814: TestPoint, TestPoint:TestPoint_Pad_D1.0mm, symbol Connector:TestPoint
- renumbered C802 to C801, C801 to C802, C805 to C804, C804 to C805, J802 to J801, J801 to J802, TP815 to TP801, TP809 to TP802, TP802 to TP803, TP812 to TP804, TP804 to TP805, TP805 to TP806, TP806 to TP807
Other:
- moved on the sheet: TP801
