File: Power.kicad_sch (KiCad schematic)
At the start: 25 parts, among them U201 AP62200WU-7, U202 TLV75733PDRV

Commit message: refactor: change motor output, renamed power nets
Connections:
- net P_VIN: now also C207.1, C208.1, C209.1, D203.1 (K), U201.3 (IN); no longer D203.2 (A), TP201.1
- net D_ADC1_CH11 renamed D_ADC2_CH13
- removed net VBAT: C207.1, C208.1, C209.1, D203.1 (K), R205.1, U201.3 (IN)
- new net P_VBAT: D203.2 (A), R205.1, TP201.1
Changed lines of the file:
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@@
 	)
 	(junction
-		(at 116.84 68.58)
-		(diameter 0)
-		(color 0 0 0 0)
-	)
-	(junction
 		(at 111.76 69.85)
 		(diameter 0)
@@
 	)
 	(junction
+		(at 118.11 68.58)
+		(diameter 0)
+		(color 0 0 0 0)
+	)
+	(junction
 		(at 194.31 86.36)
 		(diameter 0)
@@
 	)
 	(junction
-		(at 111.76 68.58)
-		(diameter 0)
-		(color 0 0 0 0)
-	)
-	(junction
 		(at 199.39 133.35)
 		(diameter 0)
@@
 	(wire
 		(pts
-			(xy 116.84 68.58) (xy 120.65 68.58)
-		)
-		(stroke
-			(width 0)
-			(type default)
-		)
-	)
-	(wire
-		(pts
-			(xy 83.82 118.11) (xy 83.82 120.65)
+			(xy 83.82 133.35) (xy 83.82 134.62)
 		)
 		(stroke
@@
 	(wire
 		(pts
-			(xy 83.82 133.35) (xy 83.82 134.62)
+			(xy 129.54 85.09) (xy 144.78 85.09)
 		)
 		(stroke
@@
 	(wire
 		(pts
-			(xy 129.54 85.09) (xy 144.78 85.09)
+			(xy 129.54 68.58) (xy 137.16 68.58)
 		)
 		(stroke
@@
 	(wire
 		(pts
-			(xy 129.54 68.58) (xy 137.16 68.58)
+			(xy 177.8 83.82) (xy 177.8 86.36)
 		)
 		(stroke
@@
 	(wire
 		(pts
-			(xy 177.8 83.82) (xy 177.8 86.36)
+			(xy 118.11 68.58) (xy 120.65 68.58)
 		)
 		(stroke
@@
 	(wire
 		(pts
-			(xy 111.76 64.77) (xy 111.76 68.58)
-		)
-		(stroke
-			(width 0)
-			(type default)
-		)
-	)
-	(wire
-		(pts
 			(xy 204.47 86.36) (xy 194.31 86.36)
 		)
@@
 	(wire
 		(pts
+			(xy 90.17 118.11) (xy 83.82 118.11)
+		)
+		(stroke
+			(width 0)
+			(type default)
+		)
+	)
+	(wire
+		(pts
+			(xy 83.82 118.11) (xy 83.82 120.65)
+		)
+		(stroke
+			(width 0)
+			(type default)
+		)
+	)
+	(wire
+		(pts
 			(xy 147.32 78.74) (xy 147.32 85.09)
 		)
@@
 	(wire
 		(pts
-			(xy 111.76 68.58) (xy 116.84 68.58)
+			(xy 111.76 68.58) (xy 118.11 68.58)
 		)
 		(stroke
@@
 		)
 	)
+	(label "P_VBAT"
+		(at 90.17 118.11 180)
+		(effects
+			(font
+				(size 1.016 1.016)
+			)
+			(justify right bottom)
+		)
+	)
 	(label "D_FB"
 		(at 170.18 77.47 0)
@@
 	)
 	(label "P_VIN"
+		(at 111.76 68.58 0)
+		(effects
+			(font
+				(size 1.016 1.016)
+			)
+			(justify left bottom)
+		)
+	)
+	(label "P_VBAT"
 		(at 92.71 69.85 0)
 		(effects
@@
 		)
 	)
-	(hierarchical_label "D_ADC1_CH11"
+	(hierarchical_label "D_ADC2_CH13"
 		(shape input)
 		(at 100.33 127 0)
@@
 	(symbol
 		(lib_id "power:PWR_FLAG")
-		(at 116.84 68.58 0)
+		(at 118.11 68.58 0)
 		(unit 1)
 		(body_style 1)
@@
 		(fields_autoplaced yes)
 		(property "Reference" "#FLG0203"
-			(at 116.84 66.675 0)
+			(at 118.11 66.675 0)
 			(hide yes)
 			(show_name no)
@@
 		)
 		(property "Value" "PWR_FLAG"
-			(at 116.84 63.5 0)
+			(at 118.11 63.5 0)
 			(hide yes)
 			(show_name no)
@@
 		)
 		(property "Footprint" ""
-			(at 116.84 68.58 0)
+			(at 118.11 68.58 0)
 			(hide yes)
 			(show_name no)
@@
 		)
 		(property "Datasheet" ""
-			(at 116.84 68.58 0)
+			(at 118.11 68.58 0)
 			(hide yes)
 			(show_name no)
@@
 		)
 		(property "Description" "Special symbol for telling ERC where power comes from"
-			(at 116.84 68.58 0)
+			(at 118.11 68.58 0)
 			(hide yes)
 			(show_name no)
@@
 	)
 	(symbol
-		(lib_id "power:VDD")
-		(at 111.76 64.77 0)
-		(unit 1)
-		(body_style 1)
-		(exclude_from_sim no)
-		(in_bom yes)
-		(on_board yes)
-		(in_pos_files yes)
-		(dnp no)
-		(property "Reference" "#PWR0204"
-			(at 111.76 68.58 0)
-			(hide yes)
-			(show_name no)
-			(do_not_autoplace no)
-			(effects
-				(font
-					(size 1.27 1.27)
-				)
-			)
-		)
-		(property "Value" "VBAT"
-			(at 111.76 60.96 0)
-			(show_name no)
-			(do_not_autoplace no)
-			(effects
-				(font
-					(size 1.27 1.27)
-				)
-			)
-		)
-		(property "Footprint" ""
-			(at 111.76 64.77 0)
-			(hide yes)
-			(show_name no)
-			(do_not_autoplace no)
-			(effects
-				(font
-					(size 1.27 1.27)
-				)
-			)
-		)
-		(property "Datasheet" ""
-			(at 111.76 64.77 0)
-			(hide yes)
-			(show_name no)
-			(do_not_autoplace no)
-			(effects
-				(font
-					(size 1.27 1.27)
-				)
-			)
-		)
-		(property "Description" "Power symbol creates a global label with name \"VDD\""
-			(at 111.76 64.77 0)
-			(hide yes)
-			(show_name no)
-			(do_not_autoplace no)
-			(effects
-				(font
-					(size 1.27 1.27)
-				)
-			)
-		)
-		(pin "1"
-		)
-		(instances
-			(project "FeroFlyF405"
-				(path "/8fea5468-8d8d-4bdb-afc0-e65b62c92669/8c352998-3abb-4e27-b22f-570d9eb08340"
-					(reference "#PWR0204")
-					(unit 1)
-				)
-			)
-		)
-	)
-	(symbol
 		(lib_id "Device:LED_Small")
 		(at 217.17 120.65 180)
@@
 		)
 	)
-	(symbol
-		(lib_id "power:VDD")
-		(at 83.82 118.11 0)
-		(unit 1)
-		(body_style 1)
-		(exclude_from_sim no)
-		(in_bom yes)
-		(on_board yes)
-		(in_pos_files yes)
-		(dnp no)
-		(property "Reference" "#PWR0205"
-			(at 83.82 121.92 0)
-			(hide yes)
-			(show_name no)
-			(do_not_autoplace no)
-			(effects
-				(font
-					(size 1.27 1.27)
-				)
-			)
-		)
-		(property "Value" "VBAT"
-			(at 83.82 114.3 0)
-			(show_name no)
-			(do_not_autoplace no)
-			(effects
-				(font
-					(size 1.27 1.27)
-				)
-			)
-		)
-		(property "Footprint" ""
-			(at 83.82 118.11 0)
-			(hide yes)
-			(show_name no)
-			(do_not_autoplace no)
-			(effects
-				(font
-					(size 1.27 1.27)
-				)
-			)
-		)
-		(property "Datasheet" ""
-			(at 83.82 118.11 0)
-			(hide yes)
-			(show_name no)
-			(do_not_autoplace no)
-			(effects
-				(font
-					(size 1.27 1.27)
-				)
-			)
-		)
-		(property "Description" "Power symbol creates a global label with name \"VDD\""
-			(at 83.82 118.11 0)
-			(hide yes)
-			(show_name no)
-			(do_not_autoplace no)
-			(effects
-				(font
-					(size 1.27 1.27)
-				)
-			)
-		)
-		(pin "1"
-		)
-		(instances
-			(project "FeroFlyF405"
-				(path "/8fea5468-8d8d-4bdb-afc0-e65b62c92669/8c352998-3abb-4e27-b22f-570d9eb08340"
-					(reference "#PWR0205")
-					(unit 1)
-				)
-			)
-		)
-	)
 	(group "TLV75733PDRV 5V to 3V3 LDO"
 		(lib_id "LDO:TLV75733PDRV 5V to 3V3 LDO")
@@
 			"586f5feb-deab-4caf-be0a-bb50dda0a7cb" "59393135-ec82-42aa-806c-64f4a4e9a5ba"
 			"5af383f5-026f-4ad0-8372-ac2e10e87989" "5bcefc9e-4033-4012-a7a6-c2eb75c9e0ec"
-			"6020b4cb-d6d9-4f7e-b6e5-a303e21da4e2" "6321c341-3fe6-417e-a32d-ddaced3692a1"
-			"63b08ea2-8204-45a8-aa9c-b9e1540141e9" "6bd96ba4-4928-42b8-8389-19d9b3e9f5f4"
-			"6c6e0c14-afad-477b-89cf-35a4bf20de09" "72aae39b-b449-4208-b708-4474f59e5d38"
-			"7b16d398-0ef6-40a8-b305-f76fdd29cfa2" "7fdcef17-c78e-4adf-a190-b8209437da3c"
-			"83e9b82c-6d2b-4257-b4f0-6710951e7258" "8624ad8b-a793-41a1-a271-db488002b5e1"
-			"86ef56f9-4600-44f7-9efe-7db11e620cfd" "896974be-c101-46e1-848e-896c5c5972df"
-			"8cf8a9d2-6695-441e-b895-c6b04eebd1aa" "8ea2e0a8-f82b-4189-94a0-8c2a91d4ee14"
-			"92c0fe5f-0d0b-4035-abd4-f5d8176b2d88" "97588cf4-3083-4d00-b06a-c70ae79744ce"
-			"9b1ff41b-2146-4023-8d95-5ad25ec27cbd" "9b693a1f-c7a9-49ec-b957-c236d91e763d"
-			"9dd698e1-a52c-4bd1-99b9-ca5372d5fcfa" "9e4a0fc1-6f3a-4aab-a969-24e533e0eabd"
-			"9e6f00c7-dee3-4c55-9a6a-3cd6308a7dbe" "9f1a245d-22b3-4cc1-901d-0f291c370392"
-			"9fb258b8-345b-467f-99e3-995613ebe33a" "a046420f-a375-4fba-974a-956e16746f44"
+			"6321c341-3fe6-417e-a32d-ddaced3692a1" "63b08ea2-8204-45a8-aa9c-b9e1540141e9"
+			"6bd96ba4-4928-42b8-8389-19d9b3e9f5f4" "6c6e0c14-afad-477b-89cf-35a4bf20de09"
+			"72aae39b-b449-4208-b708-4474f59e5d38" "7b16d398-0ef6-40a8-b305-f76fdd29cfa2"
+			"7fdcef17-c78e-4adf-a190-b8209437da3c" "83e9b82c-6d2b-4257-b4f0-6710951e7258"
+			"8624ad8b-a793-41a1-a271-db488002b5e1" "86ef56f9-4600-44f7-9efe-7db11e620cfd"
+			"896974be-c101-46e1-848e-896c5c5972df" "8cf8a9d2-6695-441e-b895-c6b04eebd1aa"
+			"8ea2e0a8-f82b-4189-94a0-8c2a91d4ee14" "92c0fe5f-0d0b-4035-abd4-f5d8176b2d88"
+			"97588cf4-3083-4d00-b06a-c70ae79744ce" "9b1ff41b-2146-4023-8d95-5ad25ec27cbd"
+			"9b693a1f-c7a9-49ec-b957-c236d91e763d" "9dd698e1-a52c-4bd1-99b9-ca5372d5fcfa"
+			"9e4a0fc1-6f3a-4aab-a969-24e533e0eabd" "9e6f00c7-dee3-4c55-9a6a-3cd6308a7dbe"
+			"9f1a245d-22b3-4cc1-901d-0f291c370392" "9fb258b8-345b-467f-99e3-995613ebe33a"
+			"a046420f-a375-4fba-974a-956e16746f44" "a158cd65-e1f4-40d8-843e-1f18678caf85"
 			"a1ae669e-dd45-4aa2-94e0-d62b0e1e0d7a" "a75fef34-be9b-4ba3-9bfd-016d06be7fd3"
 			"a781f3ea-f70d-44db-92ce-141e55ac24b6" "a7e4f5ea-172e-4210-bd75-e42807492c0c"
@@
 			"c5cd9225-a551-4e2c-a262-dfaf42769e9a" "c770a358-cb4b-4542-8fd3-c4c053a13e04"
 			"c7e5e63b-96e4-4ef1-9db3-74fe50e9e239" "c9c8c8c2-f100-4fe2-a893-d8349ddb23d8"
-			"cb69951e-8d4b-4384-a499-060ffd25ec0f" "d3423552-d9f5-4872-bcd3-b4102146770e"
-			"d3a81c59-3707-4619-8f85-6f817c813872" "d6dbb5b7-1e3f-45ce-a86d-51af64d69b8b"
-			"dedaccec-d3be-430a-bfbc-919d465999e9" "e3656e8e-59da-417d-8b5c-f01a0110e814"
-			"e90ac307-c53b-4cbe-90a5-27190df05d13" "ea14a82b-0f41-4992-9ef6-6da046ea358b"
+			"cb69951e-8d4b-4384-a499-060ffd25ec0f" "d3a81c59-3707-4619-8f85-6f817c813872"
+			"d6dbb5b7-1e3f-45ce-a86d-51af64d69b8b" "dedaccec-d3be-430a-bfbc-919d465999e9"
+			"e3656e8e-59da-417d-8b5c-f01a0110e814" "e90ac307-c53b-4cbe-90a5-27190df05d13"
 			"f29f2c4d-a10c-4c4b-a193-2342874acf47" "f5d1a81d-9ed5-4e18-9f04-f328a214fdd3"
 			"f615d222-bfb7-4113-8175-28f27fe33a16" "f94d6fab-cbe6-44e1-b623-4c9c644ceedc"
 			"fa31e384-77f5-4c8b-91a5-f2c0bd51bbf3" "fce33441-6ee5-4a40-9fb3-45b146c10b10"
-			"fdac7a27-42fa-4e41-91be-923aa246afb6" "fe1c4aa9-7bea-46d9-923a-8c1d23726854"
+			"fe1c4aa9-7bea-46d9-923a-8c1d23726854"
 		)
 	)
