File: peripherals 2.kicad_sch (KiCad schematic)
At the start: 14 parts, among them J601 SM04B-GHS-TB(LF)(SN), U601 SN65HVD230DR

Commit message: feat: add layout notes and net labels
Parts:
- R605: footprint Resistor_SMD:R_0603_1608Metric_Pad0.98x0.95mm_HandSolder -> Resistor_SMD:R_1206_3216Metric_Pad1.30x1.75mm_HandSolder; MPN CR0603-FX-1200ELF -> CR1206-FX-1200ELF
Connections:
- net CAN-: now reaches D603.1 (K), J601.3 (Pin_3), R605.2, U601.6 (CANL)
- net CAN+: now reaches D603.2 (K), J601.2 (Pin_2), JP601.1 (A), U601.7 (CANH)
Changed lines of the file:
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@@
+		)
+	)
+	(table
+		(column_count 1)
+		(border
+			(external yes)
+			(header yes)
+			(stroke
+				(width 0)
+				(type solid)
+			)
+		)
+		(separators
+			(rows yes)
+			(cols yes)
+			(stroke
+				(width 0)
+				(type solid)
+			)
+		)
+		(column_widths 14.605)
+		(row_heights 6.35 2.54 2.54 2.54 2.54)
+		(cells
+			(table_cell "SILK SCREEN TEXT ORDER Pin 1 to 4"
+				(exclude_from_sim no)
+				(at 144.78 101.6 0)
+				(size 14.605 6.35)
+				(margins 0.9525 0.9525 0.9525 0.9525)
+				(span 1 1)
+				(fill
+					(type none)
+				)
+				(effects
+					(font
+						(size 1.016 1.016)
+					)
+					(justify top)
+				)
+			)
+			(table_cell "5V"
+				(exclude_from_sim no)
+				(at 144.78 107.95 0)
+				(size 14.605 2.54)
+				(margins 0.9525 0.9525 0.9525 0.9525)
+				(span 1 1)
+				(fill
+					(type none)
+				)
+				(effects
+					(font
+						(size 1.27 1.27)
+					)
+					(justify top)
+				)
+			)
+			(table_cell "CANH"
+				(exclude_from_sim no)
+				(at 144.78 110.49 0)
+				(size 14.605 2.54)
+				(margins 0.9525 0.9525 0.9525 0.9525)
+				(span 1 1)
+				(fill
+					(type none)
+				)
+				(effects
+					(font
+						(size 1.27 1.27)
+					)
+					(justify top)
+				)
+			)
+			(table_cell "CANL"
+				(exclude_from_sim no)
+				(at 144.78 113.03 0)
+				(size 14.605 2.54)
+				(margins 0.9525 0.9525 0.9525 0.9525)
+				(span 1 1)
+				(fill
+					(type none)
+				)
+				(effects
+					(font
+						(size 1.27 1.27)
+					)
+					(justify top)
+				)
+			)
+			(table_cell "GND"
+				(exclude_from_sim no)
+				(at 144.78 115.57 0)
+				(size 14.605 2.54)
+				(margins 0.9525 0.9525 0.9525 0.9525)
+				(span 1 1)
+				(fill
+					(type none)
+				)
+				(effects
+					(font
+						(size 1.27 1.27)
+					)
+					(justify top)
+				)
+			)
+		)
+	)
+	(label "CAN+"
+		(at 96.52 93.98 0)
+		(effects
+			(font
+				(size 1.27 1.27)
+			)
+			(justify left bottom)
 		)
 	)
@@
 			(font
 				(size 0.762 0.762)
+			)
+			(justify left bottom)
+		)
+	)
+	(label "CAN-"
+		(at 96.52 96.52 0)
+		(effects
+			(font
+				(size 1.27 1.27)
 			)
 			(justify left bottom)
@@
 			)
 		)
-		(property "Footprint" "Resistor_SMD:R_0603_1608Metric_Pad0.98x0.95mm_HandSolder"
+		(property "Footprint" "Resistor_SMD:R_1206_3216Metric_Pad1.30x1.75mm_HandSolder"
 			(at 114.3 88.9 0)
 			(hide yes)
@@
 			)
 		)
-		(property "MPN" "CR0603-FX-1200ELF"
+		(property "MPN" "CR1206-FX-1200ELF"
 			(at 114.3 88.9 0)
 			(hide yes)
@@
 			(at 114.3 88.9 0)
 			(hide yes)
-			(show_name no)
-			(do_not_autoplace no)
-			(effects
-				(font
-					(size 1.27 1.27)
-				)
-			)
-		)
-		(property "MANUFACTURER" ""
-			(at 114.3 88.9 0)
-			(hide yes)

Commit message: refactor: change name from FeroFly405 to FeroFlyF405
Other:
- title: FeroFly405 -> FeroFlyF405
Changed lines of the file:
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@@
 	(paper "A4")
 	(title_block
-		(title "FeroFly405")
+		(title "FeroFlyF405")
 		(date "2026-07-22")
 		(rev "1")
-		(comment 3 "GitHub: https://github.com/Ozonised/FeroFly405")
+		(comment 3 "GitHub: https://github.com/Ozonised/FeroFlyF405")
 		(comment 4 "Designed by: Farhan Khan")
 	)
@@
 		)
 		(instances
-			(project "FeroFly"
+			(project "FeroFlyF405"
 				(path "/8fea5468-8d8d-4bdb-afc0-e65b62c92669/2db1372a-2ed6-420c-af8b-d4f9c1346569/367b3cbf-5e59-446e-ac2c-a19d2fd73a05"
 					(reference "R605")
@@
 		)
 		(instances
-			(project "FeroFly"
+			(project "FeroFlyF405"
 				(path "/8fea5468-8d8d-4bdb-afc0-e65b62c92669/2db1372a-2ed6-420c-af8b-d4f9c1346569/367b3cbf-5e59-446e-ac2c-a19d2fd73a05"
 					(reference "#PWR0608")
@@
 		)
 		(instances
-			(project "FeroFly"
+			(project "FeroFlyF405"
 				(path "/8fea5468-8d8d-4bdb-afc0-e65b62c92669/2db1372a-2ed6-420c-af8b-d4f9c1346569/367b3cbf-5e59-446e-ac2c-a19d2fd73a05"
 					(reference "#PWR0606")
@@
 		)
 		(instances
-			(project "FeroFly"
+			(project "FeroFlyF405"
 				(path "/8fea5468-8d8d-4bdb-afc0-e65b62c92669/2db1372a-2ed6-420c-af8b-d4f9c1346569/367b3cbf-5e59-446e-ac2c-a19d2fd73a05"
 					(reference "#PWR0607")
@@
 		)
 		(instances
-			(project "FeroFly"
+			(project "FeroFlyF405"
 				(path "/8fea5468-8d8d-4bdb-afc0-e65b62c92669/2db1372a-2ed6-420c-af8b-d4f9c1346569/367b3cbf-5e59-446e-ac2c-a19d2fd73a05"
 					(reference "D603")
@@
 		)
 		(instances
-			(project "FeroFly"
+			(project "FeroFlyF405"
 				(path "/8fea5468-8d8d-4bdb-afc0-e65b62c92669/2db1372a-2ed6-420c-af8b-d4f9c1346569/367b3cbf-5e59-446e-ac2c-a19d2fd73a05"
 					(reference "C602")
@@
 		)
 		(instances
-			(project "FeroFly"
+			(project "FeroFlyF405"
 				(path "/8fea5468-8d8d-4bdb-afc0-e65b62c92669/2db1372a-2ed6-420c-af8b-d4f9c1346569/367b3cbf-5e59-446e-ac2c-a19d2fd73a05"
 					(reference "JP601")
@@
 		)
 		(instances
-			(project "FeroFly"
+			(project "FeroFlyF405"
 				(path "/8fea5468-8d8d-4bdb-afc0-e65b62c92669/2db1372a-2ed6-420c-af8b-d4f9c1346569/367b3cbf-5e59-446e-ac2c-a19d2fd73a05"
 					(reference "R602")
@@
 		)
 		(instances
-			(project "FeroFly"
+			(project "FeroFlyF405"
 				(path "/8fea5468-8d8d-4bdb-afc0-e65b62c92669/2db1372a-2ed6-420c-af8b-d4f9c1346569/367b3cbf-5e59-446e-ac2c-a19d2fd73a05"
 					(reference "#PWR0602")
@@
 		)
 		(instances
-			(project "FeroFly"
+			(project "FeroFlyF405"
 				(path "/8fea5468-8d8d-4bdb-afc0-e65b62c92669/2db1372a-2ed6-420c-af8b-d4f9c1346569/367b3cbf-5e59-446e-ac2c-a19d2fd73a05"
 					(reference "R604")
@@
 		)
 		(instances
-			(project "FeroFly"
+			(project "FeroFlyF405"
 				(path "/8fea5468-8d8d-4bdb-afc0-e65b62c92669/2db1372a-2ed6-420c-af8b-d4f9c1346569/367b3cbf-5e59-446e-ac2c-a19d2fd73a05"
 					(reference "D602")
@@
 		)
 		(instances
-			(project "FeroFly"
+			(project "FeroFlyF405"
 				(path "/8fea5468-8d8d-4bdb-afc0-e65b62c92669/2db1372a-2ed6-420c-af8b-d4f9c1346569/367b3cbf-5e59-446e-ac2c-a19d2fd73a05"
 					(reference "#PWR0605")
@@
 		)
 		(instances
-			(project "FeroFly"
+			(project "FeroFlyF405"
 				(path "/8fea5468-8d8d-4bdb-afc0-e65b62c92669/2db1372a-2ed6-420c-af8b-d4f9c1346569/367b3cbf-5e59-446e-ac2c-a19d2fd73a05"
 					(reference "#PWR0604")
@@
 		)
 		(instances
-			(project "FeroFly"
+			(project "FeroFlyF405"
 				(path "/8fea5468-8d8d-4bdb-afc0-e65b62c92669/2db1372a-2ed6-420c-af8b-d4f9c1346569/367b3cbf-5e59-446e-ac2c-a19d2fd73a05"
 					(reference "J601")
@@
 		)
 		(instances
-			(project "FeroFly"
+			(project "FeroFlyF405"
 				(path "/8fea5468-8d8d-4bdb-afc0-e65b62c92669/2db1372a-2ed6-420c-af8b-d4f9c1346569/367b3cbf-5e59-446e-ac2c-a19d2fd73a05"
 					(reference "U601")
@@
 		)
 		(instances
-			(project "FeroFly"
+			(project "FeroFlyF405"
 				(path "/8fea5468-8d8d-4bdb-afc0-e65b62c92669/2db1372a-2ed6-420c-af8b-d4f9c1346569/367b3cbf-5e59-446e-ac2c-a19d2fd73a05"
 					(reference "R603")
@@
 		)
 		(instances
-			(project "FeroFly"
+			(project "FeroFlyF405"
 				(path "/8fea5468-8d8d-4bdb-afc0-e65b62c92669/2db1372a-2ed6-420c-af8b-d4f9c1346569/367b3cbf-5e59-446e-ac2c-a19d2fd73a05"
 					(reference "C603")
@@
 		)
 		(instances
-			(project "FeroFly"
+			(project "FeroFlyF405"
 				(path "/8fea5468-8d8d-4bdb-afc0-e65b62c92669/2db1372a-2ed6-420c-af8b-d4f9c1346569/367b3cbf-5e59-446e-ac2c-a19d2fd73a05"
 					(reference "C601")
@@
 		)
 		(instances
-			(project "FeroFly"
+			(project "FeroFlyF405"
 				(path "/8fea5468-8d8d-4bdb-afc0-e65b62c92669/2db1372a-2ed6-420c-af8b-d4f9c1346569/367b3cbf-5e59-446e-ac2c-a19d2fd73a05"
 					(reference "#PWR0601")
@@
 		)
 		(instances
-			(project "FeroFly"
+			(project "FeroFlyF405"
 				(path "/8fea5468-8d8d-4bdb-afc0-e65b62c92669/2db1372a-2ed6-420c-af8b-d4f9c1346569/367b3cbf-5e59-446e-ac2c-a19d2fd73a05"
 					(reference "#PWR0603")
@@
 		)
 		(instances
-			(project "FeroFly"
+			(project "FeroFlyF405"
 				(path "/8fea5468-8d8d-4bdb-afc0-e65b62c92669/2db1372a-2ed6-420c-af8b-d4f9c1346569/367b3cbf-5e59-446e-ac2c-a19d2fd73a05"
 					(reference "D601")
@@
 		)
 		(instances
-			(project "FeroFly"
+			(project "FeroFlyF405"
 				(path "/8fea5468-8d8d-4bdb-afc0-e65b62c92669/2db1372a-2ed6-420c-af8b-d4f9c1346569/367b3cbf-5e59-446e-ac2c-a19d2fd73a05"
 					(reference "R601")

Commit message: refactor(schematic): assign net classes and fix USB net label assingment
Connections:
- net D_CANTR: now reaches JP601.2 (B), R605.1
Changed lines of the file:
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@@
+		)
+	)
+	(label "D_CANTR"
+		(at 107.95 81.28 0)
+		(effects
+			(font
+				(size 0.762 0.762)
+			)
+			(justify left bottom)
 		)
 	)

Commit message: fix: RSD CAN connection
Connections:
- net CAN+: now also D603.1 (K); no longer D603.2 (K)
- net CAN-: now also D603.2 (K); no longer D603.1 (K)
Changed lines of the file:
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@@
-	)
-	(junction
-		(at 119.38 96.52)
-		(diameter 0)
-		(color 0 0 0 0)
 	)
 	(junction
@@
 	)
 	(junction
-		(at 124.46 93.98)
+		(at 124.46 96.52)
+		(diameter 0)
+		(color 0 0 0 0)
+	)
+	(junction
+		(at 119.38 93.98)
 		(diameter 0)
 		(color 0 0 0 0)
@@
 	(wire
 		(pts
-			(xy 119.38 96.52) (xy 119.38 97.79)
+			(xy 119.38 93.98) (xy 119.38 97.79)
 		)
 		(stroke
@@
 	(wire
 		(pts
-			(xy 114.3 96.52) (xy 119.38 96.52)
-		)
-		(stroke
-			(width 0)
-			(type default)
-		)
-	)
-	(wire
-		(pts
 			(xy 95.25 93.98) (xy 105.41 93.98)
 		)
@@
 	(wire
 		(pts
-			(xy 124.46 93.98) (xy 135.89 93.98)
+			(xy 105.41 93.98) (xy 119.38 93.98)
+		)
+		(stroke
+			(width 0)
+			(type default)
+		)
+	)
+	(wire
+		(pts
+			(xy 124.46 96.52) (xy 124.46 97.79)
 		)
 		(stroke
@@
 	(wire
 		(pts
-			(xy 105.41 93.98) (xy 124.46 93.98)
-		)
-		(stroke
-			(width 0)
-			(type default)
-		)
-	)
-	(wire
-		(pts
 			(xy 114.3 91.44) (xy 114.3 96.52)
 		)
@@
 	(wire
 		(pts
+			(xy 124.46 96.52) (xy 135.89 96.52)
+		)
+		(stroke
+			(width 0)
+			(type default)
+		)
+	)
+	(wire
+		(pts
 			(xy 105.41 81.28) (xy 114.3 81.28)
 		)
@@
 	(wire
 		(pts
+			(xy 119.38 93.98) (xy 135.89 93.98)
+		)
+		(stroke
+			(width 0)
+			(type default)
+		)
+	)
+	(wire
+		(pts
 			(xy 76.2 83.82) (xy 76.2 85.09)
 		)
@@
 	(wire
 		(pts
-			(xy 119.38 96.52) (xy 135.89 96.52)
+			(xy 114.3 96.52) (xy 124.46 96.52)
 		)
 		(stroke
@@
 		)
 		(stroke
-			(width 0)
-			(type default)
-		)
-	)
-	(wire
-		(pts
-			(xy 124.46 93.98) (xy 124.46 97.79)
-		)
-		(stroke

Commit message: fix: change footprint for IO & LDO
Parts:
- D603: footprint Package_TO_SOT_SMD:SOT-23_Handsoldering -> Package_TO_SOT_SMD:SOT-23
Changed lines of the file:
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@@
 			)
 		)
-		(property "Footprint" "Package_TO_SOT_SMD:SOT-23_Handsoldering"
+		(property "Footprint" "Package_TO_SOT_SMD:SOT-23"
 			(at 127.635 104.14 0)
 			(hide yes)

Commit message: refactor: rename net
Connections:
- net D_CANTR renamed CAN+R
Changed lines of the file:
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@@
 		)
 	)
-	(label "D_CANTR"
+	(label "CAN+R"
 		(at 107.95 81.28 0)
 		(effects
