File: FeroFlyF405.kicad_pcb (KiCad board)
At the start: 4 copper layers, 50 x 65 mm, 148 parts, among them J302 SM04B-GHS-TB(LF)(SN), J601 SM04B-GHS-TB(LF)(SN), J801 SM06B-GHS-TB(LF)(SN), J802 SM04B-GHS-TB(LF)(SN), J803 SM04B-GHS-TB(LF)(SN), J804 SM04B-GHS-TB(LF)(SN), J805 SM06B-GHS-TB(LF)(SN), J901 Conn_01x03_Pin, J902 Conn_01x03_Pin, J903 Conn_01x03_Pin, J904 Conn_01x03_Pin, J905 Conn_01x03_Pin, J906 Conn_01x03_Pin, J907 Conn_01x03_Pin, J908 Conn_01x03_Pin, J909 Conn_01x03_Pin, J910 Conn_01x03_Pin, J911 Conn_01x03_Pin, J912 Conn_01x03_Pin, J913 12402012E212A, J914 SM04B-GHS-TB(LF)(SN), SW301 SW_Push, SW302 SW_Push, U201 AP62200WU-7, U202 TLV75733PDRV, U301 STM32F405RGTx, U501 LSM6DSL, U502 DPS368, U601 SN65HVD230DR, U901 USBLC6-2P6, Y301 24MHz

Commit message: feat: add silkscreen & board characteristics and update gerbers
Parts:
- moved D601 17.0 mm to (158.9, 132.4)
- moved D602 17.0 mm to (163.1, 132.4)
- moved R601 17.0 mm to (160.9, 132.4)
- moved R605 17.0 mm to (155.0, 128.1)
- moved R901 17.0 mm to (170.6, 79.9)
- moved TP802 17.0 mm to (157.5, 77.7)
- moved C201 17.0 mm to (138.6, 126.0)
- moved C202 17.0 mm to (125.8, 121.2)
- moved C203 17.0 mm to (136.4, 126.0)
- moved C204 17.0 mm to (133.8, 128.5)
- moved C205 17.0 mm to (138.4, 119.0)
- moved C206 17.0 mm to (129.7, 121.2)
- moved C207 17.0 mm to (124.8, 115.3)
- moved C208 17.0 mm to (127.8, 115.3)
- moved C209 17.0 mm to (130.6, 115.3)
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Other:
- board text added: "S 5V G"

Commit message: feat: add series resistor for PINIO
Parts:
- added R801: 330, Resistor_SMD:R_0603_1608Metric_Pad0.98x0.95mm_HandSolder, B.Cu at (137.6, 74.2)
- added R802: 330, Resistor_SMD:R_0603_1608Metric_Pad0.98x0.95mm_HandSolder, B.Cu at (136.0, 75.8)
- renumbered G to TP803
Connections:
- J804 pad 2: /IO/D_PINIO0 -> /IO/IO1/D_PINIO0R
- J804 pad 3: /IO/D_PINIO1 -> /IO/IO1/D_PINIO1R
Routing:
- net /IO/IO1/D_PINIO1R: track 0.00 -> 6.06 mm, vias 0 -> 1
- net /IO/D_PINIO1: track 26.2 -> 20.2 mm, vias 2 -> 1
- net /IO/IO1/D_PINIO0R: track 0.00 -> 4.60 mm, vias 0 -> 1
- net /IO/D_PINIO0: track 27.1 -> 22.5 mm, vias 2 -> 1
