File: MCU.kicad_sch (KiCad schematic)
At the start: 35 parts, among them J302 SM04B-GHS-TB(LF)(SN), SW301 SW_Push, SW302 SW_Push, U301 STM32F405RGTx, Y301 24MHz

Commit message: refactor: change tim5 ch 1 label to ch 2
Connections:
- net D_TIM5_CH1 renamed D_TIM5_CH2
Changed lines of the file:
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@@
 		)
 	)
-	(hierarchical_label "D_TIM5_CH1"
+	(hierarchical_label "D_TIM5_CH2"
 		(shape bidirectional)
 		(at 185.42 76.2 0)
@@
 		)
 		(property "Description" "Unpolarized capacitor, small symbol"
-			(at 109.22 55.88 0)
+			(at 109.22 66.04 0)
 			(hide yes)
 			(show_name no)
@@
 		)
 		(property "Description" "Unpolarized capacitor, small symbol"
-			(at 177.8 55.88 0)
+			(at 177.8 66.04 0)
 			(hide yes)
 			(show_name no)
@@
 		)
 		(property "Description" "Unpolarized capacitor, small symbol"
-			(at 118.11 55.88 0)
+			(at 118.11 66.04 0)
 			(hide yes)
 			(show_name no)
@@
 		)
 		(property "Description" "Unpolarized capacitor, small symbol"
-			(at 63.5 101.6 0)
+			(at 63.5 111.76 0)
 			(hide yes)
 			(show_name no)
@@
 		)
 		(property "Description" "Unpolarized capacitor, small symbol"
-			(at 100.33 55.88 0)
+			(at 100.33 66.04 0)
 			(hide yes)
 			(show_name no)
@@
 		)
 		(property "Description" "Unpolarized capacitor, small symbol"
-			(at 168.91 55.88 0)
+			(at 168.91 66.04 0)
 			(hide yes)
 			(show_name no)
@@
 		)
 		(property "Description" "Unpolarized capacitor, small symbol"
-			(at 135.89 55.88 0)
+			(at 135.89 66.04 0)
 			(hide yes)
 			(show_name no)
@@
 		)
 		(property "Description" "Unpolarized capacitor, small symbol"
-			(at 96.52 96.52 0)
+			(at 96.52 106.68 0)
 			(hide yes)
 			(show_name no)
@@
 		)
 		(property "Description" "Unpolarized capacitor, small symbol"
-			(at 91.44 55.88 0)
+			(at 91.44 66.04 0)
 			(hide yes)
 			(show_name no)
@@
 		)
 		(property "Description" "Unpolarized capacitor, small symbol"
-			(at 60.96 77.47 0)
+			(at 60.96 87.63 0)
 			(hide yes)
 			(show_name no)
@@
 		)
 		(property "Description" "Unpolarized capacitor, small symbol"
-			(at 96.52 87.63 0)
+			(at 96.52 97.79 0)
 			(hide yes)
 			(show_name no)
@@
 		)
 		(property "Description" "Unpolarized capacitor, small symbol"
-			(at 118.11 147.32 0)
+			(at 118.11 157.48 0)
 			(hide yes)
 			(show_name no)
@@
 		)
 		(property "Description" "Unpolarized capacitor, small symbol"
-			(at 127 55.88 0)
+			(at 127 66.04 0)
 			(hide yes)
 			(show_name no)
@@
 		)
 		(property "Description" "Unpolarized capacitor, small symbol"
-			(at 125.73 147.32 0)
+			(at 125.73 157.48 0)
 			(hide yes)
 			(show_name no)

Commit message: fix!: change ouput 3 timer from tim4 ch4 to tim1 ch3
tim4 ch4 does not have dma. Therefore replaced it with tim1 ch3.
Connections:
- net D_TIM1_CH3: now reaches U301.43 (PA10)
- net D_TIM4_CH4: no longer names the net of U301.62 (PB9)
Changed lines of the file:
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@@
 		(title "FeroFlyF405")
 		(date "2026-07-22")
-		(rev "1")
+		(rev "1.1")
 		(comment 2 "LICENSE: CERN-OHL-S-2.0 ")
 		(comment 3 "GitHub: https://github.com/Ozonised/FeroFlyF405")
@@
 	)
 	(no_connect
-		(at 175.26 99.06)
-	)
-	(no_connect
 		(at 134.62 101.6)
 	)
@@
 	)
 	(no_connect
+		(at 175.26 139.7)
+	)
+	(no_connect
 		(at 175.26 116.84)
 	)
@@
 	(wire
 		(pts
+			(xy 175.26 99.06) (xy 185.42 99.06)
+		)
+		(stroke
+			(width 0)
+			(type default)
+		)
+	)
+	(wire
+		(pts
 			(xy 60.96 81.28) (xy 36.83 81.28)
 		)
@@
 		(pts
 			(xy 124.46 121.92) (xy 134.62 121.92)
-		)
-		(stroke
-			(width 0)
-			(type default)
-		)
-	)
-	(wire
-		(pts
-			(xy 175.26 139.7) (xy 185.42 139.7)
 		)
 		(stroke
@@
 		)
 	)
-	(hierarchical_label "D_TIM4_CH4"
+	(hierarchical_label "D_TIM1_CH3"
 		(shape bidirectional)
-		(at 185.42 139.7 0)
-		(effects
-			(font
+		(at 185.42 99.06 0)
+		(effects
+			(font
